Commit message: ongoing : change pkg name

File: RoboND-Perception-Exercises/Exercise-3/sensor_stick2/urdf/sensor_stick.gazebo.xacro (robot description, xacro)
@@ -4,5 +4,5 @@
   <gazebo>
     <plugin name="gazebo_ros_control" filename="libgazebo_ros_control.so">
-      <robotNamespace>/sensor_stick</robotNamespace>
+      <robotNamespace>/sensor_stick2</robotNamespace>
       <robotSimType>gazebo_ros_control/DefaultRobotHWSim</robotSimType>
     </plugin>

File: RoboND-Perception-Exercises/Exercise-3/sensor_stick2/urdf/sensor_stick.urdf.xacro (robot description, xacro)
@@ -1,4 +1,4 @@
 <?xml version="1.0"?>
-<robot name="sensor_stick" xmlns:xacro="http://www.ros.org/wiki/xacro">
+<robot name="sensor_stick2" xmlns:xacro="http://www.ros.org/wiki/xacro">
   <!--Define constants-->
   <xacro:property name="PI" value="3.14159"/>
@@ -12,5 +12,5 @@
   <xacro:property name="mass_camera" value="0.2" />
   <!--Import gazebo elements-->
-  <xacro:include filename="$(find sensor_stick)/urdf/sensor_stick.gazebo.xacro" />
+  <xacro:include filename="$(find sensor_stick2)/urdf/sensor_stick.gazebo.xacro" />
   <!--Links-->
   <link name="world"/>
@@ -76,5 +76,5 @@
     <origin xyz="0 0 0" rpy="0 0 0"/>
     <geometry>
-      <mesh filename="package://sensor_stick/meshes/asus_xtion.dae"/>
+      <mesh filename="package://sensor_stick2/meshes/asus_xtion.dae"/>
     </geometry>
   </visual>
