Commit message: training updated

File: RoboND-Perception-Exercises/Exercise-3/sensor_stick/urdf/sensor_stick.gazebo.xacro (robot description, xacro)
@@ -60,11 +60,13 @@
        <pointCloudTopicName>/camera/depth_registered/points</pointCloudTopicName>
        <frameName>camera_rgb_optical_frame</frameName>
-       <pointCloudCutoff>0.35</pointCloudCutoff>
+       <!-- <pointCloudCutoff>0.35</pointCloudCutoff> -->
+       <pointCloudCutoff>0.001</pointCloudCutoff>
        <pointCloudCutoffMax>4.5</pointCloudCutoffMax>
+       <!-- <pointCloudCutoffMax>300.0</pointCloudCutoffMax> -->
        <CxPrime>0</CxPrime>
        <Cx>0</Cx>
        <Cy>0</Cy>
        <focalLength>0</focalLength>
-       <hackBaseline>0</hackBaseline>
+       <hackBaseline>0.07</hackBaseline>
      </plugin>
    </sensor>

File: RoboND-Perception-Exercises/Exercise-3/sensor_stick/urdf/sensor_stick.urdf.xacro (robot description, xacro)
@@ -91,15 +91,15 @@
     <origin xyz="0 0 ${length1/2}" rpy="0 0 0"/>
   </joint>
-  <joint name="pan_joint" type="continuous">
+  <joint name="pan_joint" type="fixed">
     <parent link="link_1"/>
     <child link="link_2"/>
-    <axis xyz="0 0 1"/>
+    <!-- <axis xyz="0 0 1"/> -->
     <origin xyz="0 0 ${length1/2+length2/2}" rpy="0 0 -${pi/2}"/>
   </joint>
-  <joint name="tilt_joint" type="continuous">
+  <joint name="tilt_joint" type="fixed">
     <origin xyz="0.05 0 ${length2/2+0.02}" rpy="0 0.5 0" />
     <parent link="link_2" />
     <child link="camera_link" />
-    <axis xyz="0 1 0"/>
+    <!-- <axis xyz="0 1 0"/> -->
   </joint>
   <link name="camera_rgb_frame" />
@@ -128,5 +128,5 @@
   </joint>
   <!--Transmission and actuators-->
-  <transmission name="tran1">
+  <!-- <transmission name="tran1">
     <type>transmission_interface/SimpleTransmission</type>
     <joint name="pan_joint">
@@ -137,6 +137,6 @@
       <mechanicalReduction>1</mechanicalReduction>
     </actuator>
-  </transmission>
-  <transmission name="tran2">
+  </transmission> -->
+  <!-- <transmission name="tran2">
     <type>transmission_interface/SimpleTransmission</type>
     <joint name="tilt_joint">
@@ -147,4 +147,4 @@
       <mechanicalReduction>1</mechanicalReduction>
     </actuator>
-  </transmission>
+  </transmission> -->
 </robot>
